File: hardware/wireless_temp_sens.sch (EAGLE design)
At the start: 32 parts, among them Q1 BC550C, Q2 32.768kHz, Q3 1MHz

Commit message: update board schema
Parts:
- removed C6, C7: 30pF, rcl:C-EU025-024X044
- removed Q3: 1MHz, crystal:CRYSTALHC49S
Connections:
- net GND: no longer C6.2, C7.2
- net OSC1: no longer C6.1, Q3.2
- net OSC2: no longer C7.1, Q3.1
Changed lines of the file:
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@@
 <setting verticaltext="up"/>
 </settings>
-<grid distance="0.05" unitdist="inch" unit="inch" style="dots" multiple="1" display="yes" altdistance="0.025" altunitdist="inch" altunit="inch"/>
+<grid distance="0.1" unitdist="inch" unit="inch" style="lines" multiple="1" display="no" altdistance="0.01" altunitdist="inch" altunit="inch"/>
 <layers>
 <layer number="1" name="Top" color="4" fill="1" visible="no" active="no"/>
@@
 </classes>
 <parts>
-<part name="FRAME1" library="frames" deviceset="DINA4_L" device="" value="XBee Temp Hyd. sensor"/>
+<part name="WIRELESS_SENSOR" library="frames" deviceset="DINA4_L" device="" value="XBee Temp Hyd. sensor"/>
 <part name="SUPPLY" library="ma_libs" deviceset="3AA" device=""/>
 <part name="UC1" library="ma_libs" deviceset="S7V8" device=""/>
@@
 <part name="GND14" library="supply1" deviceset="GND" device=""/>
 <part name="Q2" library="crystal" deviceset="CRYSTAL" device="TC26H" value="32.768kHz"/>
-<part name="Q3" library="crystal" deviceset="CRYSTAL" device="HC49S" value="1MHz"/>
-<part name="GND15" library="supply1" deviceset="GND" device=""/>
-<part name="C6" library="rcl" deviceset="C-EU" device="025-024X044" value="30pF"/>
-<part name="C7" library="rcl" deviceset="C-EU" device="025-024X044" value="30pF"/>
 <part name="C8" library="rcl" deviceset="C-EU" device="025-024X044" value="30pF"/>
 <part name="C9" library="rcl" deviceset="C-EU" device="025-024X044" value="30pF"/>
@@
 </plain>
 <instances>
-<instance part="FRAME1" gate="G$1" x="0" y="0"/>
-<instance part="FRAME1" gate="G$2" x="162.56" y="0"/>
+<instance part="WIRELESS_SENSOR" gate="G$1" x="0" y="0"/>
+<instance part="WIRELESS_SENSOR" gate="G$2" x="162.56" y="0"/>
 <instance part="SUPPLY" gate="G$1" x="7.62" y="152.4" rot="R270"/>
 <instance part="UC1" gate="G$1" x="38.1" y="149.86"/>
@@
 <instance part="GND14" gate="1" x="246.38" y="45.72"/>
 <instance part="Q2" gate="G$1" x="242.57" y="125.73" rot="R180"/>
-<instance part="Q3" gate="G$1" x="213.36" y="146.05" rot="R180"/>
-<instance part="GND15" gate="1" x="213.36" y="135.89"/>
-<instance part="C6" gate="G$1" x="207.01" y="143.51"/>
-<instance part="C7" gate="G$1" x="219.71" y="143.51"/>
 <instance part="C8" gate="G$1" x="234.95" y="123.19"/>
 <instance part="C9" gate="G$1" x="248.92" y="123.19"/>
@@
 </segment>
 <segment>
-<pinref part="C6" gate="G$1" pin="2"/>
-<pinref part="GND15" gate="1" pin="GND"/>
-<wire x1="207.01" y1="138.43" x2="213.36" y2="138.43" width="0.1524" layer="91"/>
-<pinref part="C7" gate="G$1" pin="2"/>
-<wire x1="219.71" y1="138.43" x2="213.36" y2="138.43" width="0.1524" layer="91"/>
-<junction x="213.36" y="138.43"/>
-</segment>
-<segment>
 <pinref part="C8" gate="G$1" pin="2"/>
 <pinref part="GND16" gate="1" pin="GND"/>
@@
 <label x="63.5" y="106.68" size="1.016" layer="95" rot="R180" xref="yes"/>
 </segment>
-<segment>
-<pinref part="Q3" gate="G$1" pin="1"/>
-<pinref part="C7" gate="G$1" pin="1"/>
-<wire x1="215.9" y1="146.05" x2="219.71" y2="146.05" width="0.1524" layer="91"/>
-<wire x1="219.71" y1="146.05" x2="222.25" y2="146.05" width="0.1524" layer="91"/>
-<junction x="219.71" y="146.05"/>
-<label x="222.25" y="146.05" size="1.016" layer="95" xref="yes"/>
-</segment>
 </net>
 <net name="OSC1" class="0">
@@
 <label x="63.5" y="104.14" size="1.016" layer="95" rot="R180" xref="yes"/>
 </segment>
-<segment>
-<pinref part="C6" gate="G$1" pin="1"/>
-<pinref part="Q3" gate="G$1" pin="2"/>
-<wire x1="207.01" y1="146.05" x2="210.82" y2="146.05" width="0.1524" layer="91"/>
-<wire x1="207.01" y1="146.05" x2="204.47" y2="146.05" width="0.1524" layer="91"/>
-<junction x="207.01" y="146.05"/>
-<label x="204.47" y="146.05" size="1.016" layer="95" rot="R180" xref="yes"/>
-</segment>
-</net>
+</net>

Commit message: update schematic with G300 box
Parts:
- removed U$6: BS250P, ma_libs:BS250P
- added Q3: BS250, transistor-small-signal:BS250
Connections:
- removed net N$5: R9.1, U$6.D
- new net N$3: Q3.D, R9.1
- net BATTSENS: now also UC2.RB2/AN8/INT2; no longer UC2.RB1/AN10/INT1
- net BATTSEN_EN: now also UC2.RB1/AN10/INT1; no longer UC2.RB2/AN8/INT2
- net N$4: now also Q3.G; no longer U$6.G
- net V_BATT: now also Q3.S; no longer U$6.S
- net XBEE_RESET: now also UC2.RA1/AN1; no longer UC2.RA0/AN0
- net XBEE_SLEEP_RQ: now also UC2.RA0/AN0; no longer UC2.RA1/AN1
Changed lines of the file:
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@@
 <part name="C4" library="rcl" deviceset="C-EU" device="025-025X050" value="100nF"/>
 <part name="GND13" library="supply1" deviceset="GND" device=""/>
-<part name="U$6" library="ma_libs" deviceset="BS250P" device=""/>
 <part name="Q1" library="transistor-npn" deviceset="BC550*" device="" technology="C"/>
 <part name="R7" library="rcl" deviceset="R-EU_" device="0204/7" value="2k"/>
@@
 <part name="C9" library="rcl" deviceset="C-EU" device="025-024X044" value="30pF"/>
 <part name="GND16" library="supply1" deviceset="GND" device=""/>
+<part name="Q3" library="transistor-small-signal" deviceset="BS250" device=""/>
 </parts>
 <sheets>
@@
 <instance part="C4" gate="G$1" x="2.54" y="35.56"/>
 <instance part="GND13" gate="1" x="228.6" y="45.72"/>
-<instance part="U$6" gate="G$1" x="243.84" y="73.66"/>
 <instance part="Q1" gate="G$1" x="226.06" y="63.5"/>
 <instance part="R7" gate="G$1" x="218.44" y="63.5" rot="R180"/>
@@
 <instance part="C9" gate="G$1" x="248.92" y="123.19"/>
 <instance part="GND16" gate="1" x="242.57" y="115.57"/>
+<instance part="Q3" gate="1" x="243.84" y="76.2"/>
 </instances>
 <busses>
@@
 </segment>
 <segment>
+<pinref part="UC2" gate="A" pin="RA1/AN1"/>
+<wire x1="66.04" y1="119.38" x2="63.5" y2="119.38" width="0.1524" layer="91"/>
+<label x="63.5" y="119.38" size="1.016" layer="95" rot="R180" xref="yes"/>
+</segment>
+</net>
+<net name="XBEE_SLEEP_RQ" class="0">
+<segment>
+<label x="20.32" y="10.16" size="0.8128" layer="95" rot="R180" xref="yes"/>
+<pinref part="UC3" gate="G$1" pin="DTR/DI8"/>
+<wire x1="25.4" y1="10.16" x2="20.32" y2="10.16" width="0.1524" layer="91"/>
+</segment>
+<segment>
 <pinref part="UC2" gate="A" pin="RA0/AN0"/>
 <wire x1="66.04" y1="121.92" x2="63.5" y2="121.92" width="0.1524" layer="91"/>
 <label x="63.5" y="121.92" size="1.016" layer="95" rot="R180" xref="yes"/>
-</segment>
-</net>
-<net name="XBEE_SLEEP_RQ" class="0">
-<segment>
-<label x="20.32" y="10.16" size="0.8128" layer="95" rot="R180" xref="yes"/>
-<pinref part="UC3" gate="G$1" pin="DTR/DI8"/>
-<wire x1="25.4" y1="10.16" x2="20.32" y2="10.16" width="0.1524" layer="91"/>
-</segment>
-<segment>
-<pinref part="UC2" gate="A" pin="RA1/AN1"/>
-<wire x1="66.04" y1="119.38" x2="63.5" y2="119.38" width="0.1524" layer="91"/>
-<label x="63.5" y="119.38" size="1.016" layer="95" rot="R180" xref="yes"/>
 </segment>
 </net>
@@
 <pinref part="C5" gate="G$1" pin="1"/>
 <wire x1="233.68" y1="91.44" x2="233.68" y2="86.36" width="0.1524" layer="91"/>
-<pinref part="U$6" gate="G$1" pin="S"/>
-<wire x1="246.38" y1="78.74" x2="246.38" y2="91.44" width="0.1524" layer="91"/>
+<wire x1="246.38" y1="81.28" x2="246.38" y2="91.44" width="0.1524" layer="91"/>
 <wire x1="246.38" y1="91.44" x2="233.68" y2="91.44" width="0.1524" layer="91"/>
 <wire x1="233.68" y1="91.44" x2="228.6" y2="91.44" width="0.1524" layer="91"/>
@@
 <junction x="246.38" y="91.44"/>
 <label x="251.46" y="91.44" size="1.016" layer="95" xref="yes"/>
+<pinref part="Q3" gate="1" pin="S"/>
 </segment>
 </net>
@@
 </segment>
 <segment>
-<pinref part="UC2" gate="A" pin="RB2/AN8/INT2"/>
-<wire x1="66.04" y1="93.98" x2="63.5" y2="93.98" width="0.1524" layer="91"/>
-<label x="63.5" y="93.98" size="1.016" layer="95" rot="R180" xref="yes"/>
+<pinref part="UC2" gate="A" pin="RB1/AN10/INT1"/>
+<wire x1="66.04" y1="96.52" x2="63.5" y2="96.52" width="0.1524" layer="91"/>
+<label x="63.5" y="96.52" size="1.016" layer="95" rot="R180" xref="yes"/>
 </segment>
 </net>
@@
 <net name="N$4" class="0">
 <segment>
-<pinref part="U$6" gate="G$1" pin="G"/>
-<wire x1="241.3" y1="76.2" x2="233.68" y2="76.2" width="0.1524" layer="91"/>
+<wire x1="238.76" y1="76.2" x2="233.68" y2="76.2" width="0.1524" layer="91"/>
 <pinref part="C5" gate="G$1" pin="2"/>
 <wire x1="233.68" y1="76.2" x2="233.68" y2="78.74" width="0.1524" layer="91"/>
@@
 <pinref part="Q1" gate="G$1" pin="C"/>
 <wire x1="228.6" y1="76.2" x2="228.6" y2="68.58" width="0.1524" layer="91"/>
-</segment>
-</net>
-<net name="N$5" class="0">
-<segment>
-<pinref part="U$6" gate="G$1" pin="D"/>
-<pinref part="R9" gate="G$1" pin="1"/>
+<pinref part="Q3" gate="1" pin="G"/>
 </segment>
 </net>
@@
 </segment>
 <segment>
-<pinref part="UC2" gate="A" pin="RB1/AN10/INT1"/>
-<wire x1="66.04" y1="96.52" x2="63.5" y2="96.52" width="0.1524" layer="91"/>
-<label x="63.5" y="96.52" size="1.016" layer="95" rot="R180" xref="yes"/>
+<pinref part="UC2" gate="A" pin="RB2/AN8/INT2"/>
+<wire x1="66.04" y1="93.98" x2="63.5" y2="93.98" width="0.1524" layer="91"/>
+<label x="63.5" y="93.98" size="1.016" layer="95" rot="R180" xref="yes"/>
 </segment>
 </net>
@@
 </segment>
 </net>
+<net name="N$3" class="0">
+<segment>
+<pinref part="R9" gate="G$1" pin="1"/>
+<pinref part="Q3" gate="1" pin="D"/>
+<wire x1="246.38" y1="71.12" x2="246.38" y2="68.58" width="0.1524" layer="91"/>
+</segment>
+</net>

Commit message: add 2.54mm connector for I2C
Parts:
- removed UC4: HYT221, ma_libs:HYT221
- added U$1: HYT221HYT221-CON, ma_libs:HYT221HYT221-CON
Connections:
- net GND: now also U$1.GND; no longer UC4.GND
- net SCL: now also U$1.SCL; no longer UC4.SCL
- net SDA: now also U$1.SDA; no longer UC4.SDA
- net VCC: now also U$1.VDD; no longer UC4.VDD
Changed lines of the file:
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@@
 <part name="GND8" library="supply1" deviceset="GND" device=""/>
 <part name="P+6" library="supply1" deviceset="VCC" device=""/>
-<part name="UC4" library="ma_libs" deviceset="HYT221" device=""/>
 <part name="P+7" library="supply1" deviceset="VCC" device=""/>
 <part name="GND9" library="supply1" deviceset="GND" device=""/>
@@
 <part name="GND16" library="supply1" deviceset="GND" device=""/>
 <part name="Q3" library="transistor-small-signal" deviceset="BS250" device=""/>
+<part name="U$1" library="ma_libs" deviceset="HYT221" device="HYT221-CON"/>
 </parts>
 <sheets>
@@
 <instance part="GND8" gate="1" x="25.4" y="5.08"/>
 <instance part="P+6" gate="VCC" x="25.4" y="33.02"/>
-<instance part="UC4" gate="G$1" x="137.16" y="20.32" rot="R180"/>
 <instance part="P+7" gate="VCC" x="106.68" y="35.56"/>
 <instance part="GND9" gate="1" x="121.92" y="7.62"/>
@@
 <instance part="GND16" gate="1" x="242.57" y="115.57"/>
 <instance part="Q3" gate="1" x="243.84" y="76.2"/>
+<instance part="U$1" gate="G$1" x="137.16" y="20.32" rot="R180"/>
 </instances>
 <busses>
@@
 </segment>
 <segment>
-<pinref part="UC4" gate="G$1" pin="GND"/>
 <wire x1="124.46" y1="15.24" x2="121.92" y2="15.24" width="0.1524" layer="91"/>
 <pinref part="GND9" gate="1" pin="GND"/>
 <wire x1="121.92" y1="15.24" x2="121.92" y2="10.16" width="0.1524" layer="91"/>
+<pinref part="U$1" gate="G$1" pin="GND"/>
 </segment>
 <segment>
@@
 <pinref part="P+9" gate="VCC" pin="VCC"/>
 <wire x1="121.92" y1="22.86" x2="121.92" y2="17.78" width="0.1524" layer="91"/>
-<pinref part="UC4" gate="G$1" pin="VDD"/>
 <wire x1="121.92" y1="17.78" x2="124.46" y2="17.78" width="0.1524" layer="91"/>
+<pinref part="U$1" gate="G$1" pin="VDD"/>
 </segment>
 <segment>
@@
 </segment>
 <segment>
-<pinref part="UC4" gate="G$1" pin="SCL"/>
 <wire x1="124.46" y1="20.32" x2="106.68" y2="20.32" width="0.1524" layer="91"/>
 <label x="104.14" y="20.32" size="1.778" layer="95" rot="R180" xref="yes"/>
@@
 <wire x1="106.68" y1="22.86" x2="106.68" y2="20.32" width="0.1524" layer="91"/>
 <junction x="106.68" y="20.32"/>
+<pinref part="U$1" gate="G$1" pin="SCL"/>
 </segment>
 </net>
@@
 </segment>
 <segment>
-<pinref part="UC4" gate="G$1" pin="SDA"/>
 <wire x1="124.46" y1="12.7" x2="114.3" y2="12.7" width="0.1524" layer="91"/>
 <label x="104.14" y="12.7" size="1.778" layer="95" rot="R180" xref="yes"/>
@@
 <wire x1="114.3" y1="22.86" x2="114.3" y2="12.7" width="0.1524" layer="91"/>
 <junction x="114.3" y="12.7"/>
-</segment>
-</net>
+<pinref part="U$1" gate="G$1" pin="SDA"/>
+</segment>
+</net>

Commit message: update schematcks (width, drill and voltage fct emplacement
Changed lines of the file:
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@@
 <sheet>
 <plain>
-<text x="224.79" y="149.86" size="1.778" layer="91">Optional</text>
+<text x="237.49" y="137.16" size="1.778" layer="91">Optional</text>
 </plain>
 <instances>

Commit message: update resitor value or A/D conversion and update brd to remove some vias
Parts:
- R10: value 4.7k -> 2.2k
- R7: value 2k -> 10k
- R9: value 10k -> 4.7k
Changed lines of the file:
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@@
 <part name="GND13" library="supply1" deviceset="GND" device=""/>
 <part name="Q1" library="transistor-npn" deviceset="BC550*" device="" technology="C"/>
-<part name="R7" library="rcl" deviceset="R-EU_" device="0204/7" value="2k"/>
+<part name="R7" library="rcl" deviceset="R-EU_" device="0204/7" value="10k"/>
 <part name="R8" library="rcl" deviceset="R-EU_" device="0204/7" value="100k"/>
 <part name="C5" library="rcl" deviceset="C-EU" device="025-025X050" value="100pF"/>
-<part name="R9" library="rcl" deviceset="R-EU_" device="0204/7" value="10k"/>
-<part name="R10" library="rcl" deviceset="R-EU_" device="0204/7" value="4.7k"/>
+<part name="R9" library="rcl" deviceset="R-EU_" device="0204/7" value="4.7k"/>
+<part name="R10" library="rcl" deviceset="R-EU_" device="0204/7" value="2.2k"/>
 <part name="GND14" library="supply1" deviceset="GND" device=""/>
 <part name="Q2" library="crystal" deviceset="CRYSTAL" device="TC26H" value="32.768kHz"/>
